Commit message: updated directory structure

File: pyperbot_v2/snakebot_description/urdf/test_snakebot.urdf.xacro (robot description, xacro)
@@ -1,4 +1,5 @@
 <?xml version="1.0" encoding="UTF-8"?>
-<robot xmlns:xacro = "http://www.ros.org/wiki/xacro" name = "simplified_snakebot">
+<!-- Follows updated snakebot but with added inertial components-->
+<robot xmlns:xacro = "http://www.ros.org/wiki/xacro" name = "test_snakebot">
     <material name = "white">
         <color rgba = "1 1 1 1"/>
@@ -34,4 +35,9 @@
             </geometry>
         </collision>
+        <inertial>
+            <origin rpy = "0 1.5708 0" xyz = "0 0 0"/>
+            <mass value = "0.1"/>
+            <inertia ixx = "0.0001" ixy = "0" ixz = "0" iyy = "0.0001" iyz = "0" izz = "0.0001"/>
+        </inertial>
     </link>
     <joint name = "m1_joint_zero" type = "prismatic">
@@ -75,4 +81,9 @@
             </geometry>
         </collision>
+        <inertial>
+            <origin rpy = "0 1.5708 0" xyz = "0 0 0"/>
+            <mass value = "0.1"/>
+            <inertia ixx = "0.0001" ixy = "0" ixz = "0" iyy = "0.0001" iyz = "0" izz = "0.0001"/>
+        </inertial>
     </link>
     <joint name = "m1_third_joint" type = "fixed">
@@ -104,4 +115,9 @@
             </geometry>
         </collision>
+        <inertial>
+            <origin rpy = "0 1.5708 0" xyz = "0 0 0"/>
+            <mass value = "0.1"/>
+            <inertia ixx = "0.0001" ixy = "0" ixz = "0" iyy = "0.0001" iyz = "0" izz = "0.0001"/>
+        </inertial>
     </link>
     <link name = "m1_virtual_link"/>
@@ -153,4 +169,9 @@
             </geometry>
         </collision>
+        <inertial>
+            <origin rpy = "0 1.5708 0" xyz = "0 0 0"/>
+            <mass value = "0.1"/>
+            <inertia ixx = "0.0001" ixy = "0" ixz = "0" iyy = "0.0001" iyz = "0" izz = "0.0001"/>
+        </inertial>
     </link>
     <joint name = "m2_joint_zero" type = "prismatic">
@@ -223,4 +244,9 @@
             </geometry>
         </collision>
+        <inertial>
+            <origin rpy = "0 1.5708 0" xyz = "0 0 0"/>
+            <mass value = "0.1"/>
+            <inertia ixx = "0.0001" ixy = "0" ixz = "0" iyy = "0.0001" iyz = "0" izz = "0.0001"/>
+        </inertial>
     </link>
     <link name = "m2_virtual_link"/>
@@ -269,4 +295,9 @@
             </geometry>
         </collision>
+        <inertial>
+            <origin rpy = "0 1.5708 0" xyz = "0 0 0"/>
+            <mass value = "0.1"/>
+            <inertia ixx = "0.0001" ixy = "0" ixz = "0" iyy = "0.0001" iyz = "0" izz = "0.0001"/>
+        </inertial>
     </link>
     <joint name = "m3_joint_zero" type = "prismatic">
@@ -310,4 +341,9 @@
             </geometry>
         </collision>
+        <inertial>
+            <origin rpy = "0 1.5708 0" xyz = "0 0 0"/>
+            <mass value = "0.1"/>
+            <inertia ixx = "0.0001" ixy = "0" ixz = "0" iyy = "0.0001" iyz = "0" izz = "0.0001"/>
+        </inertial>
     </link>
     <joint name = "m3_third_joint" type = "fixed">
@@ -339,4 +375,9 @@
             </geometry>
         </collision>
+        <inertial>
+            <origin rpy = "0 1.5708 0" xyz = "0 0 0"/>
+            <mass value = "0.1"/>
+            <inertia ixx = "0.0001" ixy = "0" ixz = "0" iyy = "0.0001" iyz = "0" izz = "0.0001"/>
+        </inertial>
     </link>
     <link name = "m3_virtual_link"/>
@@ -387,4 +428,9 @@
             </geometry>
         </collision>
+        <inertial>
+            <origin rpy = "0 1.5708 0" xyz = "0 0 0"/>
+            <mass value = "0.1"/>
+            <inertia ixx = "0.0001" ixy = "0" ixz = "0" iyy = "0.0001" iyz = "0" izz = "0.0001"/>
+        </inertial>
     </link>
     <joint name = "m4_joint_zero" type = "prismatic">
@@ -428,4 +474,9 @@
             </geometry>
         </collision>
+        <inertial>
+            <origin rpy = "0 1.5708 0" xyz = "0 0 0"/>
+            <mass value = "0.1"/>
+            <inertia ixx = "0.0001" ixy = "0" ixz = "0" iyy = "0.0001" iyz = "0" izz = "0.0001"/>
+        </inertial>
     </link>
     <joint name = "m4_third_joint" type = "fixed">
@@ -457,4 +508,9 @@
             </geometry>
         </collision>
+        <inertial>
+            <origin rpy = "0 1.5708 0" xyz = "0 0 0"/>
+            <mass value = "0.1"/>
+            <inertia ixx = "0.0001" ixy = "0" ixz = "0" iyy = "0.0001" iyz = "0" izz = "0.0001"/>
+        </inertial>
     </link>
     <link name = "m4_virtual_link"/>

Commit message: included camera

File: pyperbot_v2/snakebot_description/urdf/test_snakebot.urdf.xacro (robot description, xacro)
@@ -8,4 +8,13 @@
         <color rgba = "0 0 0 1"/>
     </material>
+    <link name = "head">
+        <visual>
+            <origin rpy = "0 1.5708 0" xyz = "0 0 0"/>
+            <geometry>
+                <sphere radius = "0.05"/>
+            </geometry>
+            <material name = "black"/>
+        </visual>
+    </link>
     <!-- TODO: UPDATE TO INCLUDE FRICTION + DYNAMICS + INERTIA COMPONENTS FOR LINK-->
     <!-- MODULE ONE-->
@@ -16,9 +25,14 @@
             <origin rpy = "0 1.5708 0" xyz = "0 0 0"/>
             <geometry>
-                <cylinder radius = "0.05" length = "0.02"/>
-            </geometry>
-            <material name = "white"/>
-        </visual>
-    </link>
+                <cylinder radius = "0.05" length = "0.01"/>
+            </geometry>
+            <material name = "white"/>
+        </visual>
+    </link>
+    <joint name = "head_to_base" type = "fixed">
+        <parent link = "base_link"/>
+        <child link = "head"/>
+        <origin xyz = "-0.02 0 0"/>
+    </joint>
     <link name = "m1_bottom_bracket_one">
         <visual>
@@ -529,3 +543,17 @@
         <origin rpy = "0 0 0" xyz = "0.055 0 0"/>
     </joint>
+    <link name = "tail">
+        <visual>
+            <origin rpy = "0 1.5708 0" xyz = "0 0 0"/>
+            <geometry>
+                <cylinder radius = "0.03" length = "0.1"/>
+            </geometry>
+            <material name = "white"/>
+        </visual>
+    </link>
+    <joint name = "m4_to_tail" type = "fixed">
+        <parent link = "m4_top_bracket"/>
+        <child link = "tail"/>
+        <origin xyz = "0.0275 0 0"/>
+    </joint>
 </robot>
