Commit message: Renamed modules from 1-4 to 0-3

File: pyperbot_v2/snakebot_description/urdf/full_snakebot_no_macro.urdf.xacro (robot description, xacro)
@@ -19,4 +19,138 @@
         </visual>
     </link>
+    <!-- Module 0 -->
+    <!-- Module 0 links-->
+    <link name = "m0_base_link">
+        <visual>
+            <origin rpy = "0 1.5708 0" xyz = "0 0 0"/>
+            <geometry>
+                <cylinder radius = "0.05" length = "0.01"/>
+            </geometry>
+            <material name = "white"/>
+        </visual>
+    </link>
+    <link name = "m0_bottom_bracket">
+        <visual>
+            <origin rpy = "0 1.5708 0" xyz = "0 0 0"/>
+            <geometry>
+                <cylinder radius = "0.05" length = "0.045"/>
+            </geometry>
+            <material name = "white"/>
+        </visual>
+        <collision>
+            <origin rpy = "0 1.5708 0" xyz = "0 0 0"/>
+            <geometry>
+                <cylinder radius = "0.05" length = "0.045"/>
+            </geometry>
+        </collision>
+        <inertial>
+            <origin rpy = "0 1.5708 0" xyz = "0 0 0"/>
+            <mass value = "0.1"/>
+            <inertia ixx = "0.0001" ixy = "0" ixz = "0" iyy = "0.0001" iyz = "0" izz = "0.0001"/>
+        </inertial>
+    </link>
+    <link name = "m0_virtual_link_zero"></link>
+    <link name = "m0_virtual_link_one"></link>
+    <link name = "m0_middle_bracket">
+        <visual>
+            <origin rpy = "0 1.5708 0" xyz = "0 0 0"/>
+            <geometry>
+                <cylinder radius = "0.05" length = "0.085"/>
+            </geometry>
+            <material name = "white"/>
+        </visual>
+        <collision>
+            <origin rpy = "0 1.5708 0" xyz = "0 0 0"/>
+            <geometry>
+                <cylinder radius = "0.05" length = "0.07"/>
+            </geometry>
+        </collision>
+        <inertial>
+            <origin rpy = "0 1.5708 0" xyz = "0 0 0"/>
+            <mass value = "0.1"/>
+            <inertia ixx = "0.0001" ixy = "0" ixz = "0" iyy = "0.0001" iyz = "0" izz = "0.0001"/>
+        </inertial>
+    </link>
+    <link name = "m0_virtual_link_two"></link>
+    <link name = "m0_top_bracket">
+        <visual>
+            <origin rpy = "0 1.5708 0" xyz = "0 0 0"/>
+            <geometry>
+                <cylinder radius = "0.05" length = "0.055"/>
+            </geometry>
+            <material name = "white"/>
+        </visual>
+        <!-- Collision - only for the top half! -->
+        <collision>
+            <origin rpy = "0 1.5708 0" xyz = "0.025 0 0"/>
+            <geometry>
+                <cylinder radius = "0.05" length = "0.055"/>
+            </geometry>
+        </collision>
+        <inertial>
+            <origin rpy = "0 1.5708 0" xyz = "0 0 0"/>
+            <mass value = "0.1"/>
+            <inertia ixx = "0.0001" ixy = "0" ixz = "0" iyy = "0.0001" iyz = "0" izz = "0.0001"/>
+        </inertial>
+    </link>
+    <link name = "m0_virtual_link_three"/>
+    <!-- Module 0 joints -->
+    <!-- Head to m0 connection -->
+    <joint name = "head_to_base" type = "fixed">
+        <parent link = "m0_base_link"/>
+        <child link = "head"/>
+        <origin xyz = "-0.02 0 0"/>
+    </joint>
+    <!-- Joint 0: prismatic -->
+    <joint name = "m0_joint_zero" type = "prismatic">
+        <parent link = "m0_base_link"/>
+        <child link = "m0_bottom_bracket"/>
+        <axis xyz = "1 0 0"/>
+        <limit lower = "0" upper = "0.02" effort = "1" velocity = "0.01"/>
+        <origin rpy = "0 0 0" xyz = "0 0 0"/>
+        <dynamics damping = "0.0" friction = "0.01"/>
+    </joint>
+    <!-- Joint 1: revolute -->
+    <joint name = "m0_joint_one" type = "revolute">
+        <parent link = "m0_bottom_bracket"/>
+        <child link = "m0_virtual_link_zero"/>
+        <axis xyz = "0 0 1"/>
+        <limit lower = "-0.0873" upper = "0.0873" effort = "1" velocity = "0.01"/>
+    </joint>
+    <!-- Joint 2: revolute -->
+    <joint name = "m0_joint_two" type = "revolute">
+        <parent link = "m0_virtual_link_zero"/>
+        <child link = "m0_virtual_link_one"/>
+        <axis xyz = "1 0 0"/>
+        <limit lower = "-0.2618" upper = "0.2618" effort = "1" velocity = "0.01"/>
+        <origin xyz = "0.02 0 0"/>
+    </joint>
+    <!-- Spring-steel to cross-joint connection -->
+    <joint name = "m0_fixed_one" type = "fixed">
+        <parent link = "m0_virtual_link_one"/>
+        <child link = "m0_middle_bracket"/>
+        <origin rpy = "0 0 0" xyz = "0.045 0 0"/>
+    </joint>
+    <joint name = "m0_fixed_two" type = "fixed">
+        <parent link = "m0_middle_bracket"/>
+        <child link = "m0_virtual_link_two"/>
+        <origin rpy = "0 0 0" xyz = "0.015 0 0"/>
+    </joint>
+    <!-- Joint 3: revolute -->
+    <joint name = "m0_joint_three" type = "revolute">
+        <parent link = "m0_virtual_link_two"/>
+        <child link = "m0_virtual_link_three"/>
+        <axis xyz = "0 0 1"/>
+        <limit lower = "-0.5236" upper = "0.5236" effort = "1" velocity = "0.01"/>
+        <origin rpy = "0 0 0" xyz = "0 0 0"/>
+    </joint>
+    <!-- Joint 4: revolute -->
+    <joint name = "m0_joint_four" type = "revolute">
+        <parent link = "m0_virtual_link_three"/>
+        <child link = "m0_top_bracket"/>
+        <axis xyz = "0 1 0"/>
+        <limit lower = "-0.5236" upper = "0.5236" effort = "1" velocity = "0.01"/>
+        <origin rpy = "0 0 0" xyz = "0.055 0 0"/>
+    </joint>
     <!-- Module 1 -->
     <!-- Module 1 links-->
@@ -27,5 +161,5 @@
                 <cylinder radius = "0.05" length = "0.01"/>
             </geometry>
-            <material name = "white"/>
+            <material name = "black"/>
         </visual>
     </link>
@@ -36,5 +170,5 @@
                 <cylinder radius = "0.05" length = "0.045"/>
             </geometry>
-            <material name = "white"/>
+            <material name = "black"/>
         </visual>
         <collision>
@@ -58,5 +192,5 @@
                 <cylinder radius = "0.05" length = "0.085"/>
             </geometry>
-            <material name = "white"/>
+            <material name = "black"/>
         </visual>
         <collision>
@@ -79,5 +213,5 @@
                 <cylinder radius = "0.05" length = "0.055"/>
             </geometry>
-            <material name = "white"/>
+            <material name = "black"/>
         </visual>
         <!-- Collision - only for the top half! -->
@@ -96,9 +230,9 @@
     <link name = "m1_virtual_link_three"/>
     <!-- Module 1 joints -->
-    <!-- Head to m1 connection -->
-    <joint name = "head_to_base" type = "fixed">
-        <parent link = "m1_base_link"/>
-        <child link = "head"/>
-        <origin xyz = "-0.02 0 0"/>
+    <!-- m0 to m1 connection-->
+    <joint name = "m0_to_m1" type = "fixed">
+        <parent link = "m0_top_bracket"/>
+        <child link = "m1_base_link"/>
+        <origin xyz = "0.0275 0 0"/>
     </joint>
     <!-- Joint 0: prismatic -->
@@ -161,5 +295,5 @@
                 <cylinder radius = "0.05" length = "0.01"/>
             </geometry>
-            <material name = "black"/>
+            <material name = "white"/>
         </visual>
     </link>
@@ -170,5 +304,5 @@
                 <cylinder radius = "0.05" length = "0.045"/>
             </geometry>
-            <material name = "black"/>
+            <material name = "white"/>
         </visual>
         <collision>
@@ -192,5 +326,5 @@
                 <cylinder radius = "0.05" length = "0.085"/>
             </geometry>
-            <material name = "black"/>
+            <material name = "white"/>
         </visual>
         <collision>
@@ -213,5 +347,5 @@
                 <cylinder radius = "0.05" length = "0.055"/>
             </geometry>
-            <material name = "black"/>
+            <material name = "white"/>
         </visual>
         <!-- Collision - only for the top half! -->
@@ -295,5 +429,5 @@
                 <cylinder radius = "0.05" length = "0.01"/>
             </geometry>
-            <material name = "white"/>
+            <material name = "black"/>
         </visual>
     </link>
@@ -304,5 +438,5 @@
                 <cylinder radius = "0.05" length = "0.045"/>
             </geometry>
-            <material name = "white"/>
+            <material name = "black"/>
         </visual>
         <collision>
@@ -326,5 +460,5 @@
                 <cylinder radius = "0.05" length = "0.085"/>
             </geometry>
-            <material name = "white"/>
+            <material name = "black"/>
         </visual>
         <collision>
@@ -347,5 +481,5 @@
                 <cylinder radius = "0.05" length = "0.055"/>
             </geometry>
-            <material name = "white"/>
+            <material name = "black"/>
         </visual>
         <!-- Collision - only for the top half! -->
@@ -421,138 +555,4 @@
         <origin rpy = "0 0 0" xyz = "0.055 0 0"/>
     </joint>
-    <!-- Module 4 -->
-    <!-- Module 4 links-->
-    <link name = "m4_base_link">
-        <visual>
-            <origin rpy = "0 1.5708 0" xyz = "0 0 0"/>
-            <geometry>
-                <cylinder radius = "0.05" length = "0.01"/>
-            </geometry>
-            <material name = "black"/>
-        </visual>
-    </link>
-    <link name = "m4_bottom_bracket">
-        <visual>
-            <origin rpy = "0 1.5708 0" xyz = "0 0 0"/>
-            <geometry>
-                <cylinder radius = "0.05" length = "0.045"/>
-            </geometry>
-            <material name = "black"/>
-        </visual>
-        <collision>
-            <origin rpy = "0 1.5708 0" xyz = "0 0 0"/>
-            <geometry>
-                <cylinder radius = "0.05" length = "0.045"/>
-            </geometry>
-        </collision>
-        <inertial>
-            <origin rpy = "0 1.5708 0" xyz = "0 0 0"/>
-            <mass value = "0.1"/>
-            <inertia ixx = "0.0001" ixy = "0" ixz = "0" iyy = "0.0001" iyz = "0" izz = "0.0001"/>
-        </inertial>
-    </link>
-    <link name = "m4_virtual_link_zero"></link>
-    <link name = "m4_virtual_link_one"></link>
-    <link name = "m4_middle_bracket">
-        <visual>
-            <origin rpy = "0 1.5708 0" xyz = "0 0 0"/>
-            <geometry>
-                <cylinder radius = "0.05" length = "0.085"/>
-            </geometry>
-            <material name = "black"/>
-        </visual>
-        <collision>
-            <origin rpy = "0 1.5708 0" xyz = "0 0 0"/>
-            <geometry>
-                <cylinder radius = "0.05" length = "0.07"/>
-            </geometry>
-        </collision>
-        <inertial>
-            <origin rpy = "0 1.5708 0" xyz = "0 0 0"/>
-            <mass value = "0.1"/>
-            <inertia ixx = "0.0001" ixy = "0" ixz = "0" iyy = "0.0001" iyz = "0" izz = "0.0001"/>
-        </inertial>
-    </link>
-    <link name = "m4_virtual_link_two"></link>
-    <link name = "m4_top_bracket">
-        <visual>
-            <origin rpy = "0 1.5708 0" xyz = "0 0 0"/>
-            <geometry>
-                <cylinder radius = "0.05" length = "0.055"/>
-            </geometry>
-            <material name = "black"/>
-        </visual>
-        <!-- Collision - only for the top half! -->
-        <collision>
-            <origin rpy = "0 1.5708 0" xyz = "0.025 0 0"/>
-            <geometry>
-                <cylinder radius = "0.05" length = "0.055"/>
-            </geometry>
-        </collision>
-        <inertial>
-            <origin rpy = "0 1.5708 0" xyz = "0 0 0"/>
-            <mass value = "0.1"/>
-            <inertia ixx = "0.0001" ixy = "0" ixz = "0" iyy = "0.0001" iyz = "0" izz = "0.0001"/>
-        </inertial>
-    </link>
-    <link name = "m4_virtual_link_three"/>
-    <!-- Module 4 joints -->
-    <!-- m3 to m4 connection-->
-    <joint name = "m3_to_m4" type = "fixed">
-        <parent link = "m3_top_bracket"/>
-        <child link = "m4_base_link"/>
-        <origin xyz = "0.0275 0 0"/>
-    </joint>
-    <!-- Joint 0: prismatic -->
-    <joint name = "m4_joint_zero" type = "prismatic">
-        <parent link = "m4_base_link"/>
-        <child link = "m4_bottom_bracket"/>
-        <axis xyz = "1 0 0"/>
-        <limit lower = "0" upper = "0.02" effort = "1" velocity = "0.01"/>
-        <origin rpy = "0 0 0" xyz = "0 0 0"/>
-        <dynamics damping = "0.0" friction = "0.01"/>
-    </joint>
-    <!-- Joint 1: revolute -->
-    <joint name = "m4_joint_one" type = "revolute">
-        <parent link = "m4_bottom_bracket"/>
-        <child link = "m4_virtual_link_zero"/>
-        <axis xyz = "0 0 1"/>
-        <limit lower = "-0.0873" upper = "0.0873" effort = "1" velocity = "0.01"/>
-    </joint>
-    <!-- Joint 2: revolute -->
-    <joint name = "m4_joint_two" type = "revolute">
-        <parent link = "m4_virtual_link_zero"/>
-        <child link = "m4_virtual_link_one"/>
-        <axis xyz = "1 0 0"/>
-        <limit lower = "-0.2618" upper = "0.2618" effort = "1" velocity = "0.01"/>
-        <origin xyz = "0.02 0 0"/>
-    </joint>
-    <!-- Spring-steel to cross-joint connection -->
-    <joint name = "m4_fixed_one" type = "fixed">
-        <parent link = "m4_virtual_link_one"/>
-        <child link = "m4_middle_bracket"/>
-        <origin rpy = "0 0 0" xyz = "0.045 0 0"/>
-    </joint>
-    <joint name = "m4_fixed_two" type = "fixed">
-        <parent link = "m4_middle_bracket"/>
-        <child link = "m4_virtual_link_two"/>
-        <origin rpy = "0 0 0" xyz = "0.015 0 0"/>
-    </joint>
-    <!-- Joint 3: revolute -->
-    <joint name = "m4_joint_three" type = "revolute">
-        <parent link = "m4_virtual_link_two"/>
-        <child link = "m4_virtual_link_three"/>
-        <axis xyz = "0 0 1"/>
-        <limit lower = "-0.5236" upper = "0.5236" effort = "1" velocity = "0.01"/>
-        <origin rpy = "0 0 0" xyz = "0 0 0"/>
-    </joint>
-    <!-- Joint 4: revolute -->
-    <joint name = "m4_joint_four" type = "revolute">
-        <parent link = "m4_virtual_link_three"/>
-        <child link = "m4_top_bracket"/>
-        <axis xyz = "0 1 0"/>
-        <limit lower = "-0.5236" upper = "0.5236" effort = "1" velocity = "0.01"/>
-        <origin rpy = "0 0 0" xyz = "0.055 0 0"/>
-    </joint>
     <!-- Define tail link -->
     <link name = "tail">
@@ -565,7 +565,7 @@
         </visual>
     </link>
-    <!-- m4 to tail connection -->
-    <joint name = "m4_to_tail" type = "fixed">
-        <parent link = "m4_top_bracket"/>
+    <!-- m3 to tail connection -->
+    <joint name = "m3_to_tail" type = "fixed">
+        <parent link = "m3_top_bracket"/>
         <child link = "tail"/>
         <origin xyz = "0.0275 0 0"/>
