Commit message: updated concertina movement and manual brake

File: pyperbot_v2/snakebot_description/urdf/updated_full_snakebot_no_macro.urdf.xacro (robot description, xacro)
@@ -60,9 +60,4 @@
             </geometry>
         </collision>
-        <inertial>
-            <origin rpy = "0 1.5708 0" xyz = "0 0 0"/>
-            <mass value = "0.1"/>
-            <inertia ixx = "0.0001" ixy = "0" ixz = "0" iyy = "0.0001" iyz = "0" izz = "0.0001"/>
-        </inertial>
     </link>
     <link name = "m0_virtual_link_zero"></link>
