Commit message: updates to the snakebot to add normalisation + experiment with macros

File: pyperbot_v2/snakebot_description/urdf/full_snakebot.urdf.xacro (robot description, xacro)
@@ -9,4 +9,26 @@
         <color rgba = "0 0 0 1"/>
     </material>
+    <!-- Define head link -->
+    <!-- Define head link -->
+    <link name = "head">
+        <inertial>
+            <origin rpy = "0 1.5708 0" xyz = "0 0 0"/>
+            <mass value = "1"/>
+            <inertia ixx = "0.0001" ixy = "0" ixz = "0" iyy = "0.0001" iyz = "0" izz = "0.0001"/>
+        </inertial>
+        <visual>
+            <origin rpy = "0 1.5708 0" xyz = "0 0 0"/>
+            <geometry>
+                <sphere radius = "0.05"/>
+            </geometry>
+            <material name = "black"/>
+        </visual>
+        <collision>
+            <origin rpy = "0 1.5708 0" xyz = "0 0 0"/>
+            <geometry>
+                <sphere radius = "0.05"/>
+            </geometry>
+        </collision>
+    </link>
     <!-- Module definition -->
     <xacro:macro name = "module" params = "number color">
@@ -168,3 +190,24 @@
         <origin xyz = "0.0275 0 0"/>
     </joint>
+    <!-- Define tail link -->
+    <link name = "tail">
+        <visual>
+            <origin rpy = "0 1.5708 0" xyz = "0 0 0"/>
+            <geometry>
+                <cylinder radius = "0.03" length = "0.1"/>
+            </geometry>
+            <material name = "white"/>
+        </visual>
+        <collision>
+            <origin rpy = "0 1.5708 0" xyz = "0 0 0"/>
+            <geometry>
+                <cylinder radius = "0.03" length = "0.1"/>
+            </geometry>
+        </collision>
+        <inertial>
+            <origin rpy = "0 1.5708 0" xyz = "0 0 0"/>
+            <mass value = "1"/>
+            <inertia ixx = "0.0001" ixy = "0" ixz = "0" iyy = "0.0001" iyz = "0" izz = "0.0001"/>
+        </inertial>
+    </link>
 </robot>
