Commit message: updates to test envs and rl env

File: pyperbot_v2/snakebot_description/urdf/normalised_snakebot_no_macro.urdf.xacro (robot description, xacro)
@@ -12,4 +12,9 @@
     <!-- Define head link -->
     <link name = "head">
+        <inertial>
+            <origin rpy = "0 1.5708 0" xyz = "0 0 0"/>
+            <mass value = "1"/>
+            <inertia ixx = "0.0001" ixy = "0" ixz = "0" iyy = "0.0001" iyz = "0" izz = "0.0001"/>
+        </inertial>
         <visual>
             <origin rpy = "0 1.5708 0" xyz = "0 0 0"/>
@@ -19,4 +24,10 @@
             <material name = "black"/>
         </visual>
+        <collision>
+            <origin rpy = "0 1.5708 0" xyz = "0 0 0"/>
+            <geometry>
+                <sphere radius = "0.05"/>
+            </geometry>
+        </collision>
     </link>
     <!-- Module 0 -->
@@ -104,4 +115,5 @@
     </joint>
     <!-- Joint 0: prismatic -->
+    <!-- TODO: Check axis of motion for the prismatic joints-->
     <joint name = "m0_joint_zero" type = "prismatic">
         <parent link = "m0_base_link"/>
@@ -565,4 +577,15 @@
             <material name = "white"/>
         </visual>
+        <collision>
+            <origin rpy = "0 1.5708 0" xyz = "0 0 0"/>
+            <geometry>
+                <cylinder radius = "0.03" length = "0.1"/>
+            </geometry>
+        </collision>
+        <inertial>
+            <origin rpy = "0 1.5708 0" xyz = "0 0 0"/>
+            <mass value = "1"/>
+            <inertia ixx = "0.0001" ixy = "0" ixz = "0" iyy = "0.0001" iyz = "0" izz = "0.0001"/>
+        </inertial>
     </link>
     <!-- m3 to tail connection -->
