Commit message: updates to the server code

File: pyperbot_v2/snakebot_description/urdf/snakebot.urdf.xacro (robot description, xacro)
@@ -1,4 +1,5 @@
 <?xml version="1.0" encoding="UTF-8"?>
 <!-- Follows updated snakebot but with added inertial components-->
+<!-- NOTE: JOINT LIMITS CHANGED FROM -1 to 1 to 0 to 0.02-->
 <robot xmlns:xacro = "http://www.ros.org/wiki/xacro" name = "full_snakebot">
     <!-- Define colors -->
@@ -124,5 +125,5 @@
         <child link = "m0_virtual_link_zero"/>
         <axis xyz = "1 0 0"/>
-        <limit lower = "-0.01" upper = "0.01" effort = "10" velocity = "0.01"/>
+        <limit lower = "0" upper = "0.02" effort = "10" velocity = "0.01"/>
         <origin rpy = "0 0 0" xyz = "0 0 0"/>
     </joint>
@@ -263,5 +264,5 @@
         <child link = "m1_virtual_link_zero"/>
         <axis xyz = "1 0 0"/>
-        <limit lower = "-0.01" upper = "0.01" effort = "10" velocity = "0.01"/>
+        <limit lower = "0" upper = "0.02" effort = "10" velocity = "0.01"/>
         <origin rpy = "0 0 0" xyz = "0 0 0"/>
     </joint>
@@ -402,5 +403,5 @@
         <child link = "m2_virtual_link_zero"/>
         <axis xyz = "1 0 0"/>
-        <limit lower = "-0.01" upper = "0.01" effort = "10" velocity = "0.01"/>
+        <limit lower = "0" upper = "0.02" effort = "10" velocity = "0.01"/>
         <origin rpy = "0 0 0" xyz = "0 0 0"/>
     </joint>
@@ -541,5 +542,5 @@
         <child link = "m3_virtual_link_zero"/>
         <axis xyz = "1 0 0"/>
-        <limit lower = "-0.01" upper = "0.01" effort = "10" velocity = "0.01"/>
+        <limit lower = "0" upper = "0.02" effort = "10" velocity = "0.01"/>
         <origin rpy = "0 0 0" xyz = "0 0 0"/>
     </joint>

Commit message: Friday update

File: pyperbot_v2/snakebot_description/urdf/snakebot.urdf.xacro (robot description, xacro)
@@ -125,5 +125,5 @@
         <child link = "m0_virtual_link_zero"/>
         <axis xyz = "1 0 0"/>
-        <limit lower = "0" upper = "0.02" effort = "10" velocity = "0.01"/>
+        <limit lower = "0" upper = "0.04" effort = "10" velocity = "0.01"/>
         <origin rpy = "0 0 0" xyz = "0 0 0"/>
     </joint>
@@ -264,5 +264,5 @@
         <child link = "m1_virtual_link_zero"/>
         <axis xyz = "1 0 0"/>
-        <limit lower = "0" upper = "0.02" effort = "10" velocity = "0.01"/>
+        <limit lower = "0" upper = "0.04" effort = "10" velocity = "0.01"/>
         <origin rpy = "0 0 0" xyz = "0 0 0"/>
     </joint>
@@ -403,5 +403,5 @@
         <child link = "m2_virtual_link_zero"/>
         <axis xyz = "1 0 0"/>
-        <limit lower = "0" upper = "0.02" effort = "10" velocity = "0.01"/>
+        <limit lower = "0" upper = "0.04" effort = "10" velocity = "0.01"/>
         <origin rpy = "0 0 0" xyz = "0 0 0"/>
     </joint>
@@ -542,5 +542,5 @@
         <child link = "m3_virtual_link_zero"/>
         <axis xyz = "1 0 0"/>
-        <limit lower = "0" upper = "0.02" effort = "10" velocity = "0.01"/>
+        <limit lower = "0" upper = "0.04" effort = "10" velocity = "0.01"/>
         <origin rpy = "0 0 0" xyz = "0 0 0"/>
     </joint>

Commit message: changes to training method

File: pyperbot_v2/snakebot_description/urdf/snakebot.urdf.xacro (robot description, xacro)
@@ -125,6 +125,6 @@
         <child link = "m0_virtual_link_zero"/>
         <axis xyz = "1 0 0"/>
-        <limit lower = "0" upper = "0.04" effort = "10" velocity = "0.01"/>
-        <origin rpy = "0 0 0" xyz = "0 0 0"/>
+        <limit lower = "-0.02" upper = "0.02" effort = "10" velocity = "0.1"/>
+        <origin rpy = "0 0 0" xyz = "0.02 0 0"/>
     </joint>
     <!-- Joint 1: revolute -->
@@ -133,5 +133,5 @@
         <child link = "m0_virtual_link_one"/>
         <axis xyz = "0 0 1"/>
-        <limit lower = "-0.0873" upper = "0.0873" effort = "10" velocity = "0.01"/>
+        <limit lower = "-0.0873" upper = "0.0873" effort = "10" velocity = "0.1"/>
     </joint>
     <!-- Joint 2: revolute -->
@@ -140,5 +140,5 @@
         <child link = "m0_virtual_link_two"/>
         <axis xyz = "1 0 0"/>
-        <limit lower = "-0.2618" upper = "0.2618" effort = "10" velocity = "0.01"/>
+        <limit lower = "-0.2618" upper = "0.2618" effort = "10" velocity = "0.1"/>
         <origin xyz = "0.02 0 0"/>
     </joint>
@@ -159,5 +159,5 @@
         <child link = "m0_virtual_link_four"/>
         <axis xyz = "0 0 1"/>
-        <limit lower = "-0.5236" upper = "0.5236" effort = "10" velocity = "0.01"/>
+        <limit lower = "-0.5236" upper = "0.5236" effort = "10" velocity = "0.1"/>
         <origin rpy = "0 0 0" xyz = "0 0 0"/>
     </joint>
@@ -167,5 +167,5 @@
         <child link = "m0_top_bracket"/>
         <axis xyz = "0 1 0"/>
-        <limit lower = "-0.5236" upper = "0.5236" effort = "10" velocity = "0.01"/>
+        <limit lower = "-0.5236" upper = "0.5236" effort = "10" velocity = "0.1"/>
         <origin rpy = "0 0 0" xyz = "0.08 0 0"/>
     </joint>
@@ -264,6 +264,6 @@
         <child link = "m1_virtual_link_zero"/>
         <axis xyz = "1 0 0"/>
-        <limit lower = "0" upper = "0.04" effort = "10" velocity = "0.01"/>
-        <origin rpy = "0 0 0" xyz = "0 0 0"/>
+        <limit lower = "-0.02" upper = "0.02" effort = "10" velocity = "0.1"/>
+        <origin rpy = "0 0 0" xyz = "0.02 0 0"/>
     </joint>
     <!-- Joint 1: revolute -->
@@ -272,5 +272,5 @@
         <child link = "m1_virtual_link_one"/>
         <axis xyz = "0 0 1"/>
-        <limit lower = "-0.0873" upper = "0.0873" effort = "10" velocity = "0.01"/>
+        <limit lower = "-0.0873" upper = "0.0873" effort = "10" velocity = "0.1"/>
     </joint>
     <!-- Joint 2: revolute -->
@@ -279,5 +279,5 @@
         <child link = "m1_virtual_link_two"/>
         <axis xyz = "1 0 0"/>
-        <limit lower = "-0.2618" upper = "0.2618" effort = "10" velocity = "0.01"/>
+        <limit lower = "-0.2618" upper = "0.2618" effort = "10" velocity = "0.1"/>
         <origin xyz = "0.02 0 0"/>
     </joint>
@@ -298,5 +298,5 @@
         <child link = "m1_virtual_link_four"/>
         <axis xyz = "0 0 1"/>
-        <limit lower = "-0.5236" upper = "0.5236" effort = "10" velocity = "0.01"/>
+        <limit lower = "-0.5236" upper = "0.5236" effort = "10" velocity = "0.1"/>
         <origin rpy = "0 0 0" xyz = "0 0 0"/>
     </joint>
@@ -306,5 +306,5 @@
         <child link = "m1_top_bracket"/>
         <axis xyz = "0 1 0"/>
-        <limit lower = "-0.5236" upper = "0.5236" effort = "10" velocity = "0.01"/>
+        <limit lower = "-0.5236" upper = "0.5236" effort = "10" velocity = "0.1"/>
         <origin rpy = "0 0 0" xyz = "0.08 0 0"/>
     </joint>
@@ -403,6 +403,6 @@
         <child link = "m2_virtual_link_zero"/>
         <axis xyz = "1 0 0"/>
-        <limit lower = "0" upper = "0.04" effort = "10" velocity = "0.01"/>
-        <origin rpy = "0 0 0" xyz = "0 0 0"/>
+        <limit lower = "-0.02" upper = "0.02" effort = "10" velocity = "0.1"/>
+        <origin rpy = "0 0 0" xyz = "0.02 0 0"/>
     </joint>
     <!-- Joint 1: revolute -->
@@ -411,5 +411,5 @@
         <child link = "m2_virtual_link_one"/>
         <axis xyz = "0 0 1"/>
-        <limit lower = "-0.0873" upper = "0.0873" effort = "10" velocity = "0.01"/>
+        <limit lower = "-0.0873" upper = "0.0873" effort = "10" velocity = "0.1"/>
     </joint>
     <!-- Joint 2: revolute -->
@@ -418,5 +418,5 @@
         <child link = "m2_virtual_link_two"/>
         <axis xyz = "1 0 0"/>
-        <limit lower = "-0.2618" upper = "0.2618" effort = "10" velocity = "0.01"/>
+        <limit lower = "-0.2618" upper = "0.2618" effort = "10" velocity = "0.1"/>
         <origin xyz = "0.02 0 0"/>
     </joint>
@@ -437,5 +437,5 @@
         <child link = "m2_virtual_link_four"/>
         <axis xyz = "0 0 1"/>
-        <limit lower = "-0.5236" upper = "0.5236" effort = "10" velocity = "0.01"/>
+        <limit lower = "-0.5236" upper = "0.5236" effort = "10" velocity = "0.1"/>
         <origin rpy = "0 0 0" xyz = "0 0 0"/>
     </joint>
@@ -445,5 +445,5 @@
         <child link = "m2_top_bracket"/>
         <axis xyz = "0 1 0"/>
-        <limit lower = "-0.5236" upper = "0.5236" effort = "10" velocity = "0.01"/>
+        <limit lower = "-0.5236" upper = "0.5236" effort = "10" velocity = "0.1"/>
         <origin rpy = "0 0 0" xyz = "0.08 0 0"/>
     </joint>
@@ -542,6 +542,6 @@
         <child link = "m3_virtual_link_zero"/>
         <axis xyz = "1 0 0"/>
-        <limit lower = "0" upper = "0.04" effort = "10" velocity = "0.01"/>
-        <origin rpy = "0 0 0" xyz = "0 0 0"/>
+        <limit lower = "-0.02" upper = "0.02" effort = "10" velocity = "0.1"/>
+        <origin rpy = "0 0 0" xyz = "0.02 0 0"/>
     </joint>
     <!-- Joint 1: revolute -->
@@ -550,5 +550,5 @@
         <child link = "m3_virtual_link_one"/>
         <axis xyz = "0 0 1"/>
-        <limit lower = "-0.0873" upper = "0.0873" effort = "10" velocity = "0.01"/>
+        <limit lower = "-0.0873" upper = "0.0873" effort = "10" velocity = "0.1"/>
     </joint>
     <!-- Joint 2: revolute -->
@@ -557,5 +557,5 @@
         <child link = "m3_virtual_link_two"/>
         <axis xyz = "1 0 0"/>
-        <limit lower = "-0.2618" upper = "0.2618" effort = "10" velocity = "0.01"/>
+        <limit lower = "-0.2618" upper = "0.2618" effort = "10" velocity = "0.1"/>
         <origin xyz = "0.02 0 0"/>
     </joint>
@@ -576,5 +576,5 @@
         <child link = "m3_virtual_link_four"/>
         <axis xyz = "0 0 1"/>
-        <limit lower = "-0.5236" upper = "0.5236" effort = "10" velocity = "0.01"/>
+        <limit lower = "-0.5236" upper = "0.5236" effort = "10" velocity = "0.1"/>
         <origin rpy = "0 0 0" xyz = "0 0 0"/>
     </joint>
@@ -584,5 +584,5 @@
         <child link = "m3_top_bracket"/>
         <axis xyz = "0 1 0"/>
-        <limit lower = "-0.5236" upper = "0.5236" effort = "10" velocity = "0.01"/>
+        <limit lower = "-0.5236" upper = "0.5236" effort = "10" velocity = "0.1"/>
         <origin rpy = "0 0 0" xyz = "0.08 0 0"/>
     </joint>
